File: Multiregion-Mods-QID/1Chip-SNES/SNES_SCIC_IGR_D4_Takt.brd (EAGLE design)
At the start: 88.9 x 40.6 mm, 42 parts, among them IC1 74HC27D, IC2 74HC30D

Commit message: Update Design: - minor changes and adjustments
Parts:
- moved RES-OUT 0.32 mm to (31.8, 41.0)
- moved SRGB9 0.32 mm to (73.0, 41.0)
Other:
- outline, holes or cut-outs redrawn
- board text added: "2xR180"
- board text removed: "2xR220"
