File: Multiregion-Mods-QID/2Chip-SNES/SNES_SCIC_IGR_D4.brd (EAGLE design)
At the start: 88.9 x 37.5 mm, 27 parts, among them IC1 74HC27D, IC2 74HC30D

Commit message: Update Design: - minor changes and adjustments
Other:
- board size 88.9 x 37.5 mm -> 88.9 x 37.1 mm
- board text added: "2xR180"
- board text removed: "2xR220"
