File: RGB Bypass/SNES_RGBAmp.brd (EAGLE design)
At the start: 23.5 x 18.3 mm, 24 parts, among them U1 THS7374

Commit message: go to version 4.1
Parts:
- added U$2: THS7314, snes_div:THS7314
- moved R1 3.88 mm to (19.1, 1.59)
- moved C2 3.47 mm to (22.5, 3.65), turned to 270 degrees
- moved C1 2.25 mm to (22.5, 7.30)
- moved R32 1.75 mm to (8.41, 10.5)
- moved R22 1.43 mm to (6.03, 10.5)
- moved R11 1.24 mm to (3.97, 2.86)
- moved C11 1.24 mm to (7.78, 2.86)
- moved R12 1.11 mm to (3.65, 10.5)
- moved R21 1.02 mm to (3.97, 5.08)
- moved C21 1.02 mm to (7.78, 5.08)
- moved R31 0.85 mm to (3.97, 7.30)
- moved C31 0.85 mm to (7.78, 7.30)
- moved B 0.63 mm to (15.2, 1.91)
- moved G 0.63 mm to (13.3, 1.91)
- moved R 0.63 mm to (11.4, 1.91)
Connections:
- removed net N$12: R13.2, U1.14
- removed net N$13: R23.2, U1.13
- new net N$4: R23.2, U$2.7, U1.12
- new net N$7: R13.2, U$2.8, U1.13
- net GND: now also U$2.5, U1.1; no longer U1.4
- net N$1: now also U$2.1, U1.2; no longer U1.1
- net N$2: now also U$2.2, U1.3; no longer U1.2
- net N$8: now also U$2.6, U1.11; no longer U1.12
- net R9: now also U$2.3, U1.4; no longer U1.3
- net VCC: now also U$2.4
Routing:
- net VCC: track 40.4 -> 55.3 mm
- net N$4: track 0.00 -> 9.94 mm
- net N$13: track 8.78 -> 0.00 mm
- net N$7: track 0.00 -> 6.14 mm
- net N$12: track 4.71 -> 0.00 mm
- net R9: track 7.29 -> 10.8 mm
- net N$1: track 21.7 -> 24.4 mm
- net N$8: track 7.25 -> 9.35 mm
- net N$14: track 11.0 -> 8.99 mm
- net N$15: track 13.7 -> 12.0 mm
- net GND: track 1.37 -> 0.00 mm
- net N$3: track 9.73 -> 8.36 mm, vias 0 -> 2
- net N$16: track 16.9 -> 15.8 mm
- net N$2: track 12.4 -> 13.2 mm
Other:
- board size 23.5 x 18.3 mm -> 22.7 x 18.3 mm
- board text added: "1"
- board text added: "C2|C1"
- board text added: "SNES RGB Amp V4.1b"
- board text removed: "C1"
- board text removed: "C2"
- board text removed: "SNES RGB Amp V4.0b"

Commit message: Change resistor values
Parts:
- R12, R22, R32: value 3M6 -> 5M1
Changed lines of the file:
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@@
 <attribute name="VALUE" x="3.33375" y="5.3975" size="1.27" layer="27"/>
 </element>
-<element name="R12" library="rcl" package="R0603" value="3M6" x="3.65125" y="10.4775" smashed="yes" rot="R90"/>
-<element name="R22" library="rcl" package="R0603" value="3M6" x="6.0325" y="10.4775" smashed="yes" rot="R90"/>
-<element name="R32" library="rcl" package="R0603" value="3M6" x="8.41375" y="10.4775" smashed="yes" rot="R90"/>
+<element name="R12" library="rcl" package="R0603" value="5M1" x="3.65125" y="10.4775" smashed="yes" rot="R90"/>
+<element name="R22" library="rcl" package="R0603" value="5M1" x="6.0325" y="10.4775" smashed="yes" rot="R90"/>
+<element name="R32" library="rcl" package="R0603" value="5M1" x="8.41375" y="10.4775" smashed="yes" rot="R90"/>
 <element name="R13" library="rcl" package="R0603" value="" x="19.20875" y="12.7" smashed="yes">
 <attribute name="VALUE" x="18.57375" y="10.795" size="1.27" layer="27"/>
