File: RGB Bypass/SNES_RGBAmp_wCSYNC.brd (EAGLE design)
At the start: 23.5 x 20.6 mm, 31 parts, among them J3 SNES_MULTIAV_RGBC_ONLY, U1 THS7374

Commit message: Change resistor values
Parts:
- R12, R22, R32: value 3M6 -> 5M1
Changed lines of the file:
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@@
 <attribute name="VALUE" x="2.54" y="5.08" size="1.27" layer="27"/>
 </element>
-<element name="R12" library="rcl" package="R0603" value="3M6" x="2.8575" y="10.16" smashed="yes" rot="R90"/>
-<element name="R22" library="rcl" package="R0603" value="3M6" x="5.23875" y="10.16" smashed="yes" rot="R90"/>
-<element name="R32" library="rcl" package="R0603" value="3M6" x="7.62" y="10.16" smashed="yes" rot="R90"/>
+<element name="R12" library="rcl" package="R0603" value="5M1" x="2.8575" y="10.16" smashed="yes" rot="R90"/>
+<element name="R22" library="rcl" package="R0603" value="5M1" x="5.23875" y="10.16" smashed="yes" rot="R90"/>
+<element name="R32" library="rcl" package="R0603" value="5M1" x="7.62" y="10.16" smashed="yes" rot="R90"/>
 <element name="R13" library="rcl" package="R0603" value="" x="19.20875" y="12.7" smashed="yes">
 <attribute name="VALUE" x="18.57375" y="10.795" size="1.27" layer="27"/>
