File: Classic_MR_Boards/Switchless-Addon-1chip/SNES_AddOn1Chip.brd (EAGLE design)
At the start: 29.2 x 26.5 mm, 19 parts, among them X50 17.734M, X60 21.477M

Commit message: clean up
Routing:
- net GND: track 0.00 -> 5.71 mm
- net N$28: track 19.1 -> 19.5 mm, vias 2 -> 3
- net N$30: track 20.3 -> 20.6 mm, vias 2 -> 3
- net N$29: vias 0 -> 1
- net N$27: vias 0 -> 1
Changed lines of the file:
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@@
 <?xml version="1.0" encoding="utf-8"?>
 <!DOCTYPE eagle SYSTEM "eagle.dtd">
-<eagle version="6.5.0">
+<eagle version="7.5.0">
 <drawing>
 <settings>
@@
 <param name="mlMinCreamFrame" value="0mil"/>
 <param name="mlMaxCreamFrame" value="0mil"/>
-<param name="mlViaStopLimit" value="0mil"/>
+<param name="mlViaStopLimit" value="30mil"/>
 <param name="srRoundness" value="0"/>
 <param name="srMinRoundness" value="0mil"/>
@@
 <pass name="Default">
 <param name="RoutingGrid" value="50mil"/>
+<param name="AutoGrid" value="1"/>
+<param name="Efforts" value="0"/>
+<param name="TopRouterVariant" value="1"/>
 <param name="tpViaShape" value="round"/>
 <param name="PrefDir.1" value="|"/>
@@
 <via x="22.86" y="21.2725" extent="1-16" drill="0.6"/>
 <via x="22.86" y="24.13" extent="1-16" drill="0.6"/>
+<wire x1="21.59" y1="22.86" x2="17.78" y2="22.86" width="0.8128" layer="1"/>
+<wire x1="17.78" y1="22.86" x2="17.78" y2="20.955" width="1.6256" layer="1"/>
 </signal>
 <signal name="VCC">
@@
 <wire x1="22.5425" y1="34.605" x2="19.0525" y2="34.605" width="0.254" layer="1"/>
 <wire x1="19.0525" y1="34.605" x2="18.0975" y2="35.56" width="0.254" layer="1"/>
-<wire x1="18.0975" y1="35.56" x2="18.0975" y2="40.386" width="0.254" layer="1"/>
+<wire x1="18.0975" y1="35.56" x2="18.0975" y2="37.98" width="0.254" layer="1"/>
+<wire x1="18.0975" y1="37.98" x2="18.0975" y2="40.386" width="0.254" layer="1"/>
 <wire x1="21.5925" y1="41.275" x2="18.7325" y2="41.275" width="0.254" layer="1"/>
 <wire x1="18.7325" y1="41.275" x2="18.0975" y2="40.64" width="0.254" layer="1"/>
@@
 <wire x1="21.5925" y1="41.2725" x2="24.13" y2="38.735" width="0.254" layer="1"/>
 <wire x1="24.13" y1="38.735" x2="26.1366" y2="38.735" width="0.254" layer="1"/>
+<via x="18.0975" y="37.98" extent="1-16" drill="0.8" diameter="1.4224" alwaysstop="yes"/>
 </signal>
 <signal name="N$28">
@@
 <wire x1="20.6375" y1="33.02" x2="22.2275" y2="33.02" width="0.254" layer="1"/>
 <wire x1="22.2275" y1="33.02" x2="22.5425" y2="32.705" width="0.254" layer="1"/>
-<wire x1="20.6375" y1="33.02" x2="18.2245" y2="33.02" width="0.254" layer="1"/>
-<wire x1="18.2245" y1="33.02" x2="18.0975" y2="30.734" width="0.254" layer="1"/>
 <wire x1="21.5925" y1="29.845" x2="21.5925" y2="30.8" width="0.254" layer="1"/>
 <wire x1="21.5925" y1="30.8" x2="22.5425" y2="31.75" width="0.254" layer="1"/>
 <wire x1="22.5425" y1="31.75" x2="22.5425" y2="32.705" width="0.254" layer="1"/>
+<via x="18.0975" y="33.14" extent="1-16" drill="0.8" diameter="1.4224" alwaysstop="yes"/>
+<wire x1="18.0975" y1="30.734" x2="18.0975" y2="33.14" width="0.254" layer="1"/>
+<wire x1="20.6375" y1="33.02" x2="18.0975" y2="33.02" width="0.254" layer="1"/>
+<wire x1="18.0975" y1="33.02" x2="18.0975" y2="33.14" width="0.254" layer="1"/>
 </signal>
 <signal name="N$29">
@@
 <wire x1="35.8775" y1="34.605" x2="39.3675" y2="34.605" width="0.254" layer="1"/>
 <wire x1="39.3675" y1="34.605" x2="40.3225" y2="35.56" width="0.254" layer="1"/>
-<wire x1="40.3225" y1="35.56" x2="40.3225" y2="40.386" width="0.254" layer="1"/>
+<wire x1="40.3225" y1="35.56" x2="40.3225" y2="37.98" width="0.254" layer="1"/>
+<wire x1="40.3225" y1="37.98" x2="40.3225" y2="40.386" width="0.254" layer="1"/>
 <wire x1="36.8275" y1="41.275" x2="39.6875" y2="41.275" width="0.254" layer="1"/>
 <wire x1="39.6875" y1="41.275" x2="40.3225" y2="40.64" width="0.254" layer="1"/>
@@
 <wire x1="34.925" y1="40.005" x2="35.5575" y2="40.005" width="0.254" layer="1"/>
 <wire x1="35.5575" y1="40.005" x2="36.8275" y2="41.275" width="0.254" layer="1"/>
+<via x="40.3225" y="37.98" extent="1-16" drill="0.8" diameter="1.4224" alwaysstop="yes"/>
 </signal>
 <signal name="N$30">
@@
 <wire x1="37.7825" y1="36.195" x2="36.1975" y2="36.195" width="0.254" layer="1"/>
 <wire x1="36.1975" y1="36.195" x2="35.8775" y2="36.515" width="0.254" layer="1"/>
-<wire x1="37.7825" y1="33.02" x2="40.1955" y2="33.02" width="0.254" layer="1"/>
-<wire x1="40.1955" y1="33.02" x2="40.3225" y2="30.734" width="0.254" layer="1"/>
 <wire x1="36.8275" y1="29.845" x2="36.8275" y2="30.8" width="0.254" layer="1"/>
 <wire x1="36.8275" y1="30.8" x2="35.8775" y2="31.75" width="0.254" layer="1"/>
@@
 <wire x1="34.925" y1="36.195" x2="35.5575" y2="36.195" width="0.254" layer="1"/>
 <wire x1="35.5575" y1="36.195" x2="35.8775" y2="36.515" width="0.254" layer="1"/>
+<via x="40.3225" y="33.14" extent="1-16" drill="0.8" diameter="1.4224" alwaysstop="yes"/>
+<wire x1="40.3225" y1="30.734" x2="40.3225" y2="33.14" width="0.254" layer="1"/>
+<wire x1="37.7825" y1="33.02" x2="40.3225" y2="33.02" width="0.254" layer="1"/>
+<wire x1="40.3225" y1="33.02" x2="40.3225" y2="33.14" width="0.254" layer="1"/>
 </signal>
 <signal name="N$31">
@@
 </signal>
 </signals>
+<errors>
+</errors>
 </board>
 </drawing>
