File: digAudio/digAudio-OC0808.brd (EAGLE design)
At the start: 18.8 x 19.7 mm, 12 parts, among them IC1 DIT4096-H

Commit message: update digital audio mod incl a new no-cut design with coax
Parts:
- U$1: value PLT133/T10W -> JT_OC0808; device cs8406:PLT133/T10W -> cs8406:JT_OC-0808T*008
Connections:
- net GND: now also U$1.P$3; no longer U$1.P$1
- net N$1: now also U$1.P$1; no longer U$1.P$3
Other:
- board size 18.8 x 19.7 mm -> 18.8 x 21.5 mm
Changed lines of the file:
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@@
 <board>
 <plain>
-<wire x1="0.9525" y1="19.764375" x2="11.7475" y2="19.764375" width="0" layer="20"/>
-<wire x1="12.065" y1="19.446875" x2="12.065" y2="15.5575" width="0" layer="20"/>
+<wire x1="0.9525" y1="21.59" x2="11.7475" y2="21.59" width="0" layer="20"/>
+<wire x1="12.065" y1="21.2725" x2="12.065" y2="15.5575" width="0" layer="20"/>
 <wire x1="12.065" y1="15.5575" x2="12.065" y2="15.24" width="0" layer="20"/>
 <text x="11.668125" y="0.396875" size="1.016" layer="25" font="vector" ratio="12">DA4SNES</text>
@@
 <wire x1="12.3825" y1="15.24" x2="19.129375" y2="15.24" width="0" layer="20"/>
 <wire x1="19.129375" y1="15.24" x2="19.446875" y2="14.9225" width="0" layer="20"/>
-<wire x1="0.635" y1="19.446875" x2="0.635" y2="0.396875" width="0" layer="20"/>
+<wire x1="0.635" y1="21.2725" x2="0.635" y2="0.396875" width="0" layer="20"/>
 <wire x1="0.635" y1="0.396875" x2="0.9525" y2="0.079375" width="0" layer="20"/>
 <wire x1="0.9525" y1="0.079375" x2="19.129375" y2="0.079375" width="0" layer="20"/>
 <wire x1="19.129375" y1="0.079375" x2="19.446875" y2="0.396875" width="0" layer="20"/>
 <wire x1="19.446875" y1="0.396875" x2="19.446875" y2="14.9225" width="0" layer="20"/>
-<wire x1="0.635" y1="19.446875" x2="0.9525" y2="19.764375" width="0" layer="20"/>
-<wire x1="12.065" y1="19.446875" x2="11.7475" y2="19.764375" width="0" layer="20"/>
+<wire x1="0.635" y1="21.2725" x2="0.9525" y2="21.59" width="0" layer="20"/>
+<wire x1="12.065" y1="21.2725" x2="11.7475" y2="21.59" width="0" layer="20"/>
 <wire x1="1.825625" y1="2.936875" x2="1.825625" y2="1.74625" width="0.2032" layer="41"/>
 <wire x1="7.77875" y1="1.905" x2="7.77875" y2="2.69875" width="0.2032" layer="41"/>
@@
 <text x="1.905" y="9.36625" size="0.8128" layer="25" font="vector" ratio="15">C3</text>
 <wire x1="5.318125" y1="2.143125" x2="5.318125" y2="2.936875" width="0.2032" layer="41"/>
-<text x="2.54" y="17.700625" size="1.016" layer="25" font="vector" ratio="17">__/)__/)_</text>
+<text x="2.54" y="20.16125" size="1.016" layer="25" font="vector" ratio="17">__/)__/)_</text>
 <text x="12.065" y="8.493125" size="1.016" layer="26" font="vector" ratio="12" rot="MR0">Mapping:</text>
 <wire x1="12.303125" y1="8.09625" x2="5.476875" y2="8.09625" width="0.1524" layer="26"/>
@@
 <element name="3" library="wirepad" package="SMD0,8-1,6" value="" x="18.335625" y="5.08" smashed="yes" rot="R90"/>
 <element name="1" library="wirepad" package="SMD0,8-1,6" value="" x="18.335625" y="2.54" smashed="yes" rot="R90"/>
-<element name="U$1" library="cs8406" package="PLT133/T10W" value="PLT133/T10W" x="6.35" y="13.335" rot="MR0"/>
+<element name="U$1" library="cs8406" package="JT_OC-0808T*008" value="JT_OC0808" x="6.35" y="13.335" rot="MR0"/>
 </elements>
 <signals>
@@
 <wire x1="11.4825" y1="9.25" x2="11.4825" y2="10.2125" width="0.2032" layer="1"/>
 <wire x1="11.4825" y1="10.2125" x2="11.90625" y2="10.63625" width="0.2032" layer="1"/>
-<contactref element="U$1" pad="P$3"/>
+<contactref element="U$1" pad="P$1"/>
 <wire x1="3.81" y1="13.335" x2="5.08" y2="14.605" width="0.2032" layer="1"/>
 </signal>
@@
 <via x="1.905" y="12.065" extent="1-16" drill="0.4"/>
 <via x="2.69875" y="4.92125" extent="1-16" drill="0.4"/>
-<via x="11.7475" y="6.985" extent="1-16" drill="0.4"/>
+<via x="11.7475" y="6.905625" extent="1-16" drill="0.4"/>
+<contactref element="U$1" pad="P$3"/>
 <via x="6.19125" y="0.79375" extent="1-16" drill="0.4"/>
-<contactref element="U$1" pad="P$1"/>
 </signal>
 <signal name="VCC">
@@
 <contactref element="C1" pad="1"/>
 <contactref element="C3" pad="1"/>
-<wire x1="5.55625" y1="11.1125" x2="6.35" y2="11.90625" width="0.3048" layer="1"/>
+<wire x1="6.35" y1="11.90625" x2="5.55625" y2="11.1125" width="0.3048" layer="1"/>
 <wire x1="5.55625" y1="11.1125" x2="3.4925" y2="11.1125" width="0.3048" layer="1"/>
 <wire x1="3.4925" y1="11.1125" x2="2.54" y2="10.16" width="0.3048" layer="1"/>
@@
 <wire x1="7.14375" y1="5.55625" x2="7.5825" y2="5.1175" width="0.2032" layer="1"/>
 <wire x1="2.38125" y1="1.27" x2="2.2225" y2="1.11125" width="0.8128" layer="1"/>
+<contactref element="U$1" pad="P$2"/>
+<wire x1="6.35" y1="13.335" x2="6.35" y2="11.90625" width="0.3048" layer="1"/>
 <wire x1="10.4775" y1="1.27" x2="9.921875" y2="1.825625" width="0.4064" layer="16"/>
 <wire x1="2.2225" y1="1.11125" x2="3.571875" y2="1.11125" width="0.8128" layer="1"/>
@@
 <wire x1="5.6325" y1="2.14" x2="5.6753125" y2="2.1828125" width="0.2032" layer="1"/>
 <wire x1="5.6753125" y1="2.1828125" x2="5.9134375" y2="2.1828125" width="0.2032" layer="1"/>
-<contactref element="U$1" pad="P$2"/>
-<wire x1="6.35" y1="11.90625" x2="6.35" y2="13.335" width="0.3048" layer="1"/>
 </signal>
 <signal name="N$2">
