File: digAudio/digAudio-OC0808.sch (EAGLE design)
At the start: 12 parts, among them IC1 DIT4096-H

Commit message: update digital audio mod incl a new no-cut design with coax
Parts:
- U$1: value PLT133/T10W -> JT_OC0808; device cs8406:PLT133/T10W -> cs8406:JT_OC0808
Changed lines of the file:
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@@
 <part name="3" library="wirepad" deviceset="SMD1" device="" value=""/>
 <part name="1" library="wirepad" deviceset="SMD1" device="" value=""/>
-<part name="U$1" library="cs8406" deviceset="PLT133/T10W" device=""/>
+<part name="U$1" library="cs8406" deviceset="JT_OC0808" device=""/>
 </parts>
 <sheets>
@@
 <instance part="3" gate="G$1" x="-20.32" y="35.56"/>
 <instance part="1" gate="G$1" x="45.72" y="33.02" rot="R180"/>
-<instance part="U$1" gate="G$1" x="68.58" y="45.72"/>
+<instance part="U$1" gate="G$1" x="66.04" y="45.72"/>
 </instances>
 <busses>
