File: digAudio/digAudio-rcj-da101jc.sch (EAGLE design)
At the start: 14 parts, among them IC1 DIT4096-H

Commit message: PCB Update
Parts:
- added GND: (no value), wirepad:1,6/0,9
- added J1: (no value), jumper:SJ2W
- C3: value 10nF -> 10nF/0.1uuF
- R1: value 360 -> 347.5/57
- R2: value 91 -> 90.9/open
- VCC: device wirepad:SMD2 -> wirepad:1,6/0,9
Connections:
- new net N$12: J1.2, R2.1, U$2.3
- net GND: now also GND.P, J1.1
- net N$7: now also J1.3; no longer R2.1, U$2.3
Changed lines of the file:
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@@
 <?xml version="1.0" encoding="utf-8"?>
 <!DOCTYPE eagle SYSTEM "eagle.dtd">
-<eagle version="8.6.0">
+<eagle version="8.5.2">
 <drawing>
 <settings>
@@
 </classes>
 <parts>
-<part name="VCC" library="wirepad" library_urn="urn:adsk.eagle:library:412" deviceset="SMD2" device="" package3d_urn="urn:adsk.eagle:package:30839/1"/>
 <part name="IC1" library="texas" library_urn="urn:adsk.eagle:library:387" deviceset="DIT4192-H" device="" value="DIT4096-H"/>
 <part name="P+1" library="supply1" library_urn="urn:adsk.eagle:library:371" deviceset="VCC" device=""/>
 <part name="GND1" library="supply1" library_urn="urn:adsk.eagle:library:371" deviceset="GND" device=""/>
 <part name="GND2" library="supply1" library_urn="urn:adsk.eagle:library:371" deviceset="GND" device=""/>
-<part name="C1" library="rcl" library_urn="urn:adsk.eagle:library:334" deviceset="C-EU" device="C0603" package3d_urn="urn:adsk.eagle:package:23616/2" value="0.1uF"/>
-<part name="C2" library="rcl" library_urn="urn:adsk.eagle:library:334" deviceset="C-EU" device="C0603" package3d_urn="urn:adsk.eagle:package:23616/2" value="0.1uF"/>
-<part name="C3" library="rcl" library_urn="urn:adsk.eagle:library:334" deviceset="C-EU" device="C0603" package3d_urn="urn:adsk.eagle:package:23616/2" value="10nF"/>
+<part name="C1" library="rcl" deviceset="C-EU" device="C0603" value="0.1uF"/>
+<part name="C2" library="rcl" deviceset="C-EU" device="C0603" value="0.1uF"/>
+<part name="C3" library="rcl" deviceset="C-EU" device="C0603" value="10nF/0.1uuF"/>
 <part name="P+5" library="supply1" library_urn="urn:adsk.eagle:library:371" deviceset="VCC" device=""/>
 <part name="5" library="wirepad" library_urn="urn:adsk.eagle:library:412" deviceset="SMD1" device="" value=""/>
@@
 <part name="1" library="wirepad" library_urn="urn:adsk.eagle:library:412" deviceset="SMD1" device="" value=""/>
 <part name="U$1" library="digAudio_SNES" deviceset="RCJ_01X_SMT" device="-MODIFIED" value="RCJ-013-SMT-TR "/>
-<part name="R1" library="rcl" library_urn="urn:adsk.eagle:library:334" deviceset="R-EU_" device="R0603" package3d_urn="urn:adsk.eagle:package:23555/2" value="360"/>
-<part name="R2" library="rcl" library_urn="urn:adsk.eagle:library:334" deviceset="R-EU_" device="R0603" package3d_urn="urn:adsk.eagle:package:23555/2" value="91"/>
+<part name="R1" library="rcl" deviceset="R-EU_" device="R0603" value="347.5/57"/>
+<part name="R2" library="rcl" deviceset="R-EU_" device="R0603" value="90.9/open"/>
 <part name="U$2" library="cs8406" deviceset="DA10XJC" device=""/>
 <part name="GND3" library="supply1" library_urn="urn:adsk.eagle:library:371" deviceset="GND" device=""/>
+<part name="VCC" library="wirepad" library_urn="urn:adsk.eagle:library:412" deviceset="1,6/0,9" device="" package3d_urn="urn:adsk.eagle:package:30840/1"/>
+<part name="GND" library="wirepad" library_urn="urn:adsk.eagle:library:412" deviceset="1,6/0,9" device="" package3d_urn="urn:adsk.eagle:package:30840/1"/>
+<part name="J1" library="jumper" library_urn="urn:adsk.eagle:library:252" deviceset="SJ2W" device="" package3d_urn="urn:adsk.eagle:package:15474/1"/>
+<part name="GND4" library="supply1" library_urn="urn:adsk.eagle:library:371" deviceset="GND" device=""/>
 </parts>
 <sheets>
@@
 <wire x1="-30.48" y1="20.32" x2="-2.54" y2="20.32" width="0.1524" layer="97"/>
 <wire x1="-30.48" y1="17.526" x2="-2.54" y2="17.526" width="0.1524" layer="97"/>
-<text x="50.8" y="15.24" size="1.778" layer="97" font="vector">Boarddesign (c) 2018 by Peter Bartmann</text>
+<text x="43.18" y="10.16" size="1.778" layer="97" font="vector">Boarddesign (c) 2018 by Peter Bartmann</text>
 </plain>
 <instances>
-<instance part="VCC" gate="1" x="50.8" y="76.2"/>
 <instance part="IC1" gate="G$1" x="17.78" y="50.8"/>
 <instance part="P+1" gate="VCC" x="58.42" y="81.28"/>
@@
 <instance part="U$2" gate="G$1" x="106.68" y="35.56"/>
 <instance part="GND3" gate="1" x="86.36" y="35.56" rot="R270"/>
+<instance part="VCC" gate="1" x="50.8" y="76.2"/>
+<instance part="GND" gate="1" x="50.8" y="63.5"/>
+<instance part="J1" gate="G$1" x="68.58" y="25.4" rot="R180"/>
+<instance part="GND4" gate="1" x="68.58" y="17.78"/>
 </instances>
 <busses>
@@
 <segment>
 <pinref part="GND2" gate="1" pin="GND"/>
+<pinref part="C2" gate="G$1" pin="2"/>
 <wire x1="58.42" y1="63.5" x2="58.42" y2="60.96" width="0.1524" layer="91"/>
-<pinref part="C2" gate="G$1" pin="2"/>
 <wire x1="58.42" y1="63.5" x2="63.5" y2="63.5" width="0.1524" layer="91"/>
 <wire x1="63.5" y1="63.5" x2="73.66" y2="63.5" width="0.1524" layer="91"/>
@@
 <wire x1="63.5" y1="66.04" x2="63.5" y2="63.5" width="0.1524" layer="91"/>
 <junction x="63.5" y="63.5"/>
+<pinref part="GND" gate="1" pin="P"/>
+<wire x1="58.42" y1="63.5" x2="53.34" y2="63.5" width="0.1524" layer="91"/>
+<junction x="58.42" y="63.5"/>
 </segment>
 <segment>
@@
 <pinref part="GND3" gate="1" pin="GND"/>
 </segment>
+<segment>
+<pinref part="J1" gate="G$1" pin="1"/>
+<pinref part="GND4" gate="1" pin="GND"/>
+</segment>
 </net>
 <net name="VCC" class="0">
@@
 <pinref part="P+1" gate="VCC" pin="VCC"/>
 <wire x1="58.42" y1="78.74" x2="58.42" y2="76.2" width="0.1524" layer="91"/>
-<pinref part="VCC" gate="1" pin="P"/>
 <wire x1="53.34" y1="76.2" x2="58.42" y2="76.2" width="0.1524" layer="91"/>
 <pinref part="C2" gate="G$1" pin="1"/>
@@
 <wire x1="63.5" y1="73.66" x2="63.5" y2="76.2" width="0.1524" layer="91"/>
 <junction x="63.5" y="76.2"/>
+<pinref part="VCC" gate="1" pin="P"/>
 </segment>
 <segment>
@@
 <segment>
 <pinref part="IC1" gate="G$1" pin="TX-"/>
-<wire x1="33.02" y1="38.1" x2="58.42" y2="38.1" width="0.1524" layer="91"/>
-<wire x1="58.42" y1="38.1" x2="58.42" y2="25.4" width="0.1524" layer="91"/>
-<pinref part="R2" gate="G$1" pin="1"/>
-<wire x1="58.42" y1="25.4" x2="73.66" y2="25.4" width="0.1524" layer="91"/>
-<wire x1="73.66" y1="25.4" x2="73.66" y2="27.94" width="0.1524" layer="91"/>
-<wire x1="73.66" y1="25.4" x2="83.82" y2="25.4" width="0.1524" layer="91"/>
-<junction x="73.66" y="25.4"/>
-<wire x1="83.82" y1="25.4" x2="83.82" y2="30.48" width="0.1524" layer="91"/>
-<wire x1="88.9" y1="30.48" x2="83.82" y2="30.48" width="0.1524" layer="91"/>
-<pinref part="U$2" gate="G$1" pin="3"/>
+<wire x1="33.02" y1="38.1" x2="60.96" y2="38.1" width="0.1524" layer="91"/>
+<wire x1="60.96" y1="38.1" x2="60.96" y2="35.56" width="0.1524" layer="91"/>
+<pinref part="J1" gate="G$1" pin="3"/>
+<wire x1="60.96" y1="35.56" x2="68.58" y2="35.56" width="0.1524" layer="91"/>
+<wire x1="68.58" y1="35.56" x2="68.58" y2="30.48" width="0.1524" layer="91"/>
 </segment>
 </net>
@@
 <wire x1="132.08" y1="30.48" x2="124.46" y2="30.48" width="0.1524" layer="91"/>
 <pinref part="U$2" gate="G$1" pin="4"/>
+</segment>
+</net>
+<net name="N$12" class="0">
+<segment>
+<pinref part="U$2" gate="G$1" pin="3"/>
+<wire x1="88.9" y1="30.48" x2="83.82" y2="30.48" width="0.1524" layer="91"/>
+<wire x1="83.82" y1="25.4" x2="83.82" y2="30.48" width="0.1524" layer="91"/>
+<pinref part="R2" gate="G$1" pin="1"/>
+<wire x1="73.66" y1="25.4" x2="73.66" y2="27.94" width="0.1524" layer="91"/>
+<wire x1="73.66" y1="25.4" x2="83.82" y2="25.4" width="0.1524" layer="91"/>
+<junction x="73.66" y="25.4"/>
+<pinref part="J1" gate="G$1" pin="2"/>
 </segment>
 </net>
@@
 packages will not be understood (or retained) with this version.
 </note>
-<note version="8.4" severity="warning">
-Since Version 8.4, EAGLE supports properties for SPICE simulation.
-Probes in schematics and SPICE mapping objects found in parts and library devices
-will not be understood with this version. Update EAGLE to the latest version
-for full support of SPICE simulation.
-</note>
 </compatibility>
