File: MultiRegion_with_DeJitter_QID/SNES_MR_DeJitter_QID.brd (EAGLE design)
At the start: 85.2 x 26.4 mm, 84 parts, among them J1 SNESCART_CONN_SPARSE_4, Q31 2SC2412, U1 SuperCIC_lock, U2 uIGR, U3 EPM7032AETC44-10N, U4 74HCT2G125DP, U5 CDCE913, U6 2G17TI_DBV, U7 TLV70033, U8 TLV70018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

Commit message: update PCB design: - selectable sync level for the buffered output - video buffer for sync instead of transistor - color carrier fix applied - some GND between sub-carrier and master clock output
Parts:
- removed Q31: 2SC2412, transistor:SOT23-BEC
- removed R33: 1k, rcl:R0603
- removed R34: 10k, rcl:R0603
- removed R35: 300, rcl:R0603
- removed R36: 100, rcl:R0603
- added C91: 10u, rcl:C0603
- added C92: 0.01u, rcl:C0603
- added C93: 33u, rcl:C0805
- added C94: 22u, rcl:C0603
- added R63: 10k, rcl:R0805
- added R91: 4k7, rcl:R0603
- added R92: 2k, rcl:R0603
- added R93: 623, rcl:R0603
- added R94: 75, rcl:R0603
- added SJ63A, SJ63B, SJ93: (no value), jumper:SJ_SMALL
- added U9: TSH122ICT, st-microelectronics:SC70
- C1: device rcl:C0805 -> rcl:C0603
- moved SJ32 10.4 mm to (41.1, 1.27), turned to 180 degrees
- moved R32 4.57 mm to (43.9, 1.27), turned to 180 degrees
- moved #PALMODE_1 2.54 mm to (54.9, 23.2)
- moved C32 2.03 mm to (47.2, 1.27), turned to 0 degrees
- moved R51 0.38 mm to (55.8, 5.46)
- moved R52 0.38 mm to (55.8, 7.49)
- moved CSYNC_I1 0.25 mm to (55.4, 1.52)
Connections:
- net COLOR_SC_O renamed COLOR_SC_PCB_O
- removed net CSYNC_O_POST_Q: Q31.E, R35.1, R36.1
- removed net CSYNC_O_PRE_Q: Q31.B, R33.1, R34.1
- new net COLOR_SC_OPT_O_PRE: SJ63B.1, U3.19
- new net COLOR_SC_PCB_O_PRE: R62.1, SJ62.1, U6.4
- new net N$1: R91.2, R92.1, SJ93.1, U9.P$1
- new net N$10: R93.1, SJ93.2
- new net N$7: C94.1, U9.P$3
- new net N$8: C93.1, U9.P$4
- new net N$9: C93.2, C94.2, R94.1
- net +3V3: now also C91.1, C92.1, U9.P$5, U9.P$6
- net +5V: no longer Q31.C
- net COLOR_SC_O_PRE: now also SJ63A.2, U3.21; no longer R62.1, SJ62.1, U6.4
- net COLOR_SC_PRE: now also R63.2, SJ63A.1, SJ63B.2; no longer U3.21
- net CSYNC_O: now also R94.2; no longer R36.2
- net CSYNC_O_3V3_1: now also R91.1; no longer R33.2
- net GND: now also C91.2, C92.2, R63.1, R92.2, R93.2, U9.P$2; no longer R34.2, R35.2
Routing:
- net +5V: track 229.8 -> 187.3 mm, vias 8 -> 7
- net +3V3: track 162.1 -> 177.3 mm, vias 7 -> 8
- net SEL_SNES_1CHIP: track 4.96 -> 15.5 mm
- net N$1: track 0.00 -> 10.1 mm
- net COLOR_SC_PCB_O_PRE: track 0.00 -> 8.49 mm
- net COLOR_SC_O_PRE: track 8.49 -> 2.15 mm
- net CSYNC_O_POST_Q: track 6.22 -> 0.00 mm
- net N$9: track 0.00 -> 5.62 mm
- net COLOR_SC_OPT_O_PRE: track 0.00 -> 4.28 mm
- net CSYNC_O_PRE_Q: track 4.28 -> 0.00 mm
- net NPALMODE_1: track 14.7 -> 10.8 mm
- net N$8: track 0.00 -> 3.21 mm
- net CSYNC_O_3V3_1: track 36.1 -> 33.0 mm
- net N$7: track 0.00 -> 2.66 mm
- net N$10: track 0.00 -> 1.31 mm
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Other:
- board text added: "63"
- board text added: "Info: - Schematic and PCB design (c) 2019 - 2020 by Peter Bartmann - Design uses De-Jitter design (c) 2017-2018 by Markus Hiienkari - Design uses DFO 5V design by micro (2015)"
- board text added: "SJ"
- board text added: "SMR20200325"
- board text removed: "Info: - Schematic and PCB design (c) 2019 by Peter Bartmann - Design uses De-Jitter design (c) 2017-2018 by Markus Hiienkari - Design uses DFO 5V design by micro (2015)"
- board text removed: "SMR20190813"
